File: hardware/Feedback-Box.kicad_pcb (KiCad board)
At the start: 2 copper layers, 100 x 50 mm, 91 parts, among them J1 694106301002, J2 UJ2-BH-1-TH, J3 T821106A1S100CEU, J4 SSW-107-01-T-S, Q1 FDN340P, Q2 FDN340P, Q3 MMBT2222ALT1G, Q4 FDN340P, Q5 FDN340P, Q6 FDN340P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

Commit message: Layout revision 8B
Fixed misplaced Pin 1 locator on rear silkscreen for part J4
Other:
- board text added: "P.No. SI-FBCM01-8B © See Reverse"
- board text added: "github.com/Alarm-Siren/Feedback-Box © Nicholas Parks Young, 2020. Part Number: SI-FBCM01-8B"
- board text removed: "P.No. SI-FBCM01-8A © See Reverse"
- board text removed: "github.com/Alarm-Siren/Feedback-Box © Nicholas Parks Young, 2020. Part Number: SI-FBCM01-8A"
Changed lines of the file:
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@@
   (title_block
     (title "Feedback Box Control Module")
-    (date 2020-02-14)
-    (rev 8A)
+    (date 2020-02-25)
+    (rev 8B)
     (company "Shady Industries")
     (comment 1 "© Nicholas Parks Young, 2020. Some Rights Reserved.")
@@
   (gr_line (start 182.245 76.2) (end 182.245 74.295) (layer F.SilkS) (width 0.16))
   (gr_line (start 189.23 73.025) (end 194.31 73.025) (layer F.SilkS) (width 0.16))
-  (gr_text "P.No. SI-FBCM01-8A\n© See Reverse" (at 175.26 72.39) (layer F.SilkS)
+  (gr_text "P.No. SI-FBCM01-8B\n© See Reverse" (at 175.26 72.39) (layer F.SilkS)
     (effects (font (size 1 1) (thickness 0.16)) (justify left))
   )
@@
     (effects (font (size 1 1) (thickness 0.16)))
   )
-  (gr_text 1 (at 172.085 85.725) (layer B.SilkS)
+  (gr_text 1 (at 172.085 87.63) (layer B.SilkS)
     (effects (font (size 1 1) (thickness 0.16)) (justify mirror))
   )
@@
     (effects (font (size 1 1) (thickness 0.16)))
   )
-  (gr_text "github.com/Alarm-Siren/Feedback-Box\n© Nicholas Parks Young, 2020.\nPart Number: SI-FBCM01-8A" (at 191.77 75.565 90) (layer B.SilkS)
+  (gr_text "github.com/Alarm-Siren/Feedback-Box\n© Nicholas Parks Young, 2020.\nPart Number: SI-FBCM01-8B" (at 191.77 75.565 90) (layer B.SilkS)
     (effects (font (size 1 1) (thickness 0.16)) (justify left mirror))
   )

Commit message: Update to hardware revision 6C
Made the drill sizes for the Variable Resistors bigger, because the previous sizes where only *just* big enough.
Other:
- board text added: "P.No. SI-FBCM01-8C © See Reverse"
- board text added: "github.com/Alarm-Siren/Feedback-Box © Nicholas Parks Young, 2020. Part Number: SI-FBCM01-8C"
- board text removed: "P.No. SI-FBCM01-8B © See Reverse"
- board text removed: "github.com/Alarm-Siren/Feedback-Box © Nicholas Parks Young, 2020. Part Number: SI-FBCM01-8B"
Changed lines of the file:
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@@
   (title_block
     (title "Feedback Box Control Module")
-    (date 2020-02-25)
-    (rev 8B)
+    (date 2020-03-13)
+    (rev 8C)
     (company "Shady Industries")
     (comment 1 "© Nicholas Parks Young, 2020. Some Rights Reserved.")
@@
     (mod_text_size 1 1)
     (mod_text_width 0.16)
-    (pad_size 1 1)
-    (pad_drill 0)
+    (pad_size 1.64 1.64)
+    (pad_drill 1)
     (pad_to_mask_clearance 0.051)
     (solder_mask_min_width 0.25)
@@
     (fp_line (start -2.11 -7.305) (end -2.11 2.225) (layer F.Fab) (width 0.1))
     (fp_circle (center 1.781 -2.54) (end 3.356 -2.54) (layer F.Fab) (width 0.1))
-    (pad 1 thru_hole circle (at 0 0 270) (size 1.44 1.44) (drill 0.8) (layers *.Cu *.Mask)
+    (pad 1 thru_hole circle (at 0 0 270) (size 1.64 1.64) (drill 1) (layers *.Cu *.Mask)
       (net 6 GND))
-    (pad 2 thru_hole circle (at 5.08 -2.54 270) (size 1.44 1.44) (drill 0.8) (layers *.Cu *.Mask)
+    (pad 2 thru_hole circle (at 5.08 -2.54 270) (size 1.64 1.64) (drill 1) (layers *.Cu *.Mask)
       (net 19 "Net-(DS1-Pad3)"))
-    (pad 3 thru_hole circle (at 0 -5.08 270) (size 1.44 1.44) (drill 0.8) (layers *.Cu *.Mask)
+    (pad 3 thru_hole circle (at 0 -5.08 270) (size 1.64 1.64) (drill 1) (layers *.Cu *.Mask)
       (net 11 +5V))
     (model ${KISYS3DMOD}/Potentiometer_THT.3dshapes/Potentiometer_Bourns_3386F_Vertical.wrl
@@
       (effects (font (size 1 1) (thickness 0.15)))
     )
-    (pad 3 thru_hole circle (at 0 -5.08 90) (size 1.44 1.44) (drill 0.8) (layers *.Cu *.Mask)
+    (pad 3 thru_hole circle (at 0 -5.08 90) (size 1.64 1.64) (drill 1) (layers *.Cu *.Mask)
       (net 6 GND))
-    (pad 2 thru_hole circle (at 5.08 -2.54 90) (size 1.44 1.44) (drill 0.8) (layers *.Cu *.Mask)
+    (pad 2 thru_hole circle (at 5.08 -2.54 90) (size 1.64 1.64) (drill 1) (layers *.Cu *.Mask)
       (net 45 "Net-(Q3-Pad1)"))
-    (pad 1 thru_hole circle (at 0 0 90) (size 1.44 1.44) (drill 0.8) (layers *.Cu *.Mask)
+    (pad 1 thru_hole circle (at 0 0 90) (size 1.64 1.64) (drill 1) (layers *.Cu *.Mask)
       (net 70 SPK))
     (model ${KISYS3DMOD}/Potentiometer_THT.3dshapes/Potentiometer_Bourns_3386F_Vertical.wrl
@@
   (gr_line (start 182.245 76.2) (end 182.245 74.295) (layer F.SilkS) (width 0.16))
   (gr_line (start 189.23 73.025) (end 194.31 73.025) (layer F.SilkS) (width 0.16))
-  (gr_text "P.No. SI-FBCM01-8B\n© See Reverse" (at 175.26 72.39) (layer F.SilkS)
+  (gr_text "P.No. SI-FBCM01-8C\n© See Reverse" (at 175.26 72.39) (layer F.SilkS)
     (effects (font (size 1 1) (thickness 0.16)) (justify left))
   )
@@
     (effects (font (size 1 1) (thickness 0.16)))
   )
-  (gr_text "github.com/Alarm-Siren/Feedback-Box\n© Nicholas Parks Young, 2020.\nPart Number: SI-FBCM01-8B" (at 191.77 75.565 90) (layer B.SilkS)
+  (gr_text "github.com/Alarm-Siren/Feedback-Box\n© Nicholas Parks Young, 2020.\nPart Number: SI-FBCM01-8C" (at 191.77 75.565 90) (layer B.SilkS)
     (effects (font (size 1 1) (thickness 0.16)) (justify left mirror))
   )

Commit message: Switch R19 to 1210, 62R resistor
This allows the speaker to run at 0.35W instead of the previous 0.11W.
Parts:
- R19: value 220 -> 62; footprint Resistor_SMD:R_0603_1608Metric_Pad1.05x0.95mm_HandSolder -> Resistor_SMD:R_1210_3225Metric_Pad1.42x2.65mm_HandSolder
- moved R19 0.40 mm to (134.6, 102.9)
Routing:
- net Net-(D2-Pad1): track 11.8 -> 13.9 mm
Other:
- board text added: "P.No. SI-FBCM01-9A © See Reverse"
- board text added: "github.com/Alarm-Siren/Feedback-Box © Nicholas Parks Young, 2020. Part Number: SI-FBCM01-9A"
- board text removed: "P.No. SI-FBCM01-8C © See Reverse"
- board text removed: "github.com/Alarm-Siren/Feedback-Box © Nicholas Parks Young, 2020. Part Number: SI-FBCM01-8C"
